File: marker.kicad_sch (KiCad schematic)
At the start: 0 parts

Commit message: adding thing
Parts:
- added C1, C2, C3, C4, C5, C6, C7, C8, C9: 1nF, symbol Device:C
- added C10, C11, C13: 2.93, symbol Device:C
- added C12: 1.0uF, symbol Device:C
- added C14: 2.92, symbol Device:C
- added C15: 2.2nF, symbol Device:C
- added C16: 4.7uF, symbol Device:C
- added C17: 0.7F, symbol Device:C
- added J1: USB_A, symbol Connector:USB_A
- added L1: L, symbol Device:L
- added R1: 2R2, symbol Device:R
- added U4: nRF5340-QKxx, Package_DFN_QFN:Nordic_AQFN-94-1EP_7x7mm_P0.4mm, symbol MCU_Nordic:nRF5340-QKxx
- added Y2: Crystal, symbol Device:Crystal
Connections:
- new net: C17.1, L1.2, U4.L31 (ANT)
- new net: U4.B30 (XC2), Y2.1
- new net: U4.C31 (XC1), Y2.2
- new net: C9.2, U4.A15 (DECD)
- new net: C12.1, C15.1, U4.A27 (DECR), U4.G31 (DECRF)
- new net: J1.2 (D-), U4.B4 (D-)
- new net: J1.3 (D+), U4.B2 (D+)
- new net: C10.2, C11.2, C13.1, C14.1, U4.AA1 (NFC2/P0.03), U4.W1 (NFC1/P0.02)
- new net +5VD: R1.1
- new net GND: C1.1, C10.1, C11.1, C12.2, C13.2, C14.2, C15.2, C16.1, C17.2, C2.1, C3.1, C4.1, C5.1, C6.1, C7.1, C8.1, C9.1, U4.EP (VSS)
- new net VDD: C1.2, C2.2, C3.2, C4.2, C5.2, C6.2, C7.2, C8.2, U4.A19 (VDD), U4.AC1 (VDD), U4.AG1 (VDD), U4.AJ31 (VDD), U4.AL11 (VDD), U4.AL17 (VDD), U4.AL25 (VDD), U4.AL3 (VDD), U4.AL7 (VDD), U4.B28 (VDD), U4.B8 (VDD), U4.C1 (VDD), U4.E31 (VDD), U4.L1 (VDD), U4.N31 (VDD), U4.U1 (VDD)
- new net magic: C16.2, R1.2, U4.A5 (VBUS), U4.E1 (VDDH)

Commit message: Wasteing time
Parts:
- added H1, H10, H11, H12, H13, H14, H15, H16, H17, H18, H19, H2, H20, H21, H22, H23, H24, H25, H26, H27, H28, H29, H3, H30, H31, H32, H33, H34, H35, H36, H37, H38, H39, H4, H40, H41, H42, H43, H44, H45, H46, H5, H6, H7, H8, H9: MountingHole_Pad, MountingHole:MountingHole_2.5mm_Pad_Via, symbol Mechanical:MountingHole_Pad
- C1, C10, C11, C12, C13, C14, C15, C16, C17, C2, C3, C4, C5, C6, C7, C8, C9: footprint (none) -> Capacitor_SMD:C_0201_0603Metric
- J1: footprint (none) -> Connector_USB:USB_A_Receptacle_GCT_USB1046
- L1: footprint (none) -> Inductor_SMD:L_6.3x6.3_H3
- R1: footprint (none) -> Resistor_SMD:R_01005_0402Metric
- Y2: footprint (none) -> Crystal:Crystal_SMD_3215-2Pin_3.2x1.5mm
Connections:
- net magic: now also J1.1 (VBUS)
- net at U4.A17 (P1.13): now also H44.1
- net at U4.AB2 (AIN2/P0.06): now also H6.1
- net at U4.AD2 (AIN3/P0.07): now also H7.1
- net at U4.AE1 (TWI/P1.02): now also H33.1
- net at U4.AE31 (AIN7/P0.28): now also H28.1
- net at U4.AF2 (TWI/P1.03): now also H34.1
- net at U4.AH2 (SCK/TRACEDATA3/P0.08): now also H8.1
- net at U4.AJ1 (MOSI/TRACEDATA2/P0.09): now also H9.1
- net at U4.AK10 (IO2/P0.15): now also H15.1
- net at U4.AK12 (SCK/P0.17): now also H17.1
- net at U4.AK14 (CSN/P0.18): now also H18.1
- net at U4.AK16 (P0.20): now also H20.1
- net at U4.AK18 (P0.22): now also H22.1
- net at U4.AK2 (MISO/TRACEDATA1/P0.10): now also H1.1
- net at U4.AK20 (P0.23): now also H23.1
- net at U4.AK22 (P1.05): now also H36.1
- net at U4.AK24 (P1.07): now also H38.1
- net at U4.AK26 (P1.09): now also H40.1
- net at U4.AK28 (AIN4/P0.25): now also H25.1
- net at U4.AK30 (AIN6/P0.27): now also H27.1
- net at U4.AK4 (CSN/TRACEDATA0/P0.11): now also H11.1
- net at U4.AK6 (DCX/TRACECLK/P0.12): now also H12.1
- net at U4.AK8 (IO1/P0.14): now also H14.1
- net at U4.AL13 (P0.19): now also H19.1
- net at U4.AL15 (P0.21): now also H21.1
- net at U4.AL19 (P1.04): now also H35.1
- net at U4.AL21 (P1.06): now also H37.1
- net at U4.AL23 (P1.08): now also H39.1
- net at U4.AL27 (P0.24): now also H24.1
- net at U4.AL29 (AIN5/P0.26): now also H26.1
- net at U4.AL5 (IO0/P0.13): now also H13.1
- net at U4.AL9 (IO3/P0.16): now also H16.1
- net at U4.B14 (P1.15): now also H46.1
- net at U4.B16 (P1.14): now also H45.1
- net at U4.B18 (P1.12): now also H43.1
- net at U4.B20 (P1.11): now also H42.1
- net at U4.B22 (P0.31): now also H31.1
- net at U4.B24 (P0.30): now also H30.1
- net at U4.M2 (P1.00): now also H10.1
- net at U4.N1 (XL1/P0.00): now also H2.1
- net at U4.P2 (P1.01): now also H32.1
- net at U4.R1 (XL2/P0.01): now also H3.1
- net at U4.R31 (P1.10): now also H41.1
- net at U4.U31 (P0.29): now also H29.1
- net at U4.V2 (AIN0/P0.04): now also H4.1
- net at U4.Y2 (AIN1/P0.05): now also H5.1

Commit message: doing the things
Parts:
- removed C16: 4.7uF, Capacitor_SMD:C_0201_0603Metric, symbol Device:C
- removed C17: 0.7F, Capacitor_SMD:C_0201_0603Metric, symbol Device:C
- removed H29, H30, H31, H32, H33, H34, H35, H36, H37, H38, H39, H40, H41, H42, H43, H44, H45, H46: MountingHole_Pad, MountingHole:MountingHole_2.5mm_Pad_Via, symbol Mechanical:MountingHole_Pad
- removed J1: USB_A, Connector_USB:USB_A_Receptacle_GCT_USB1046, symbol Connector:USB_A
- removed L1: L, Inductor_SMD:L_6.3x6.3_H3, symbol Device:L
- removed R1: 2R2, Resistor_SMD:R_01005_0402Metric, symbol Device:R
- removed U4: nRF5340-QKxx, Package_DFN_QFN:Nordic_AQFN-94-1EP_7x7mm_P0.4mm, symbol MCU_Nordic:nRF5340-QKxx
- removed Y2: Crystal, Crystal:Crystal_SMD_3215-2Pin_3.2x1.5mm, symbol Device:Crystal
- added J1: 2216100001, Connector_USB:MOLEX_2216100001, symbol name:2216100001
- added R1: 1.7, Resistor_SMD:R_0201_0603Metric, symbol ScottoKeebs:Placeholder_Resistor
- added R2: 2.2, Resistor_SMD:R_0201_0603Metric, symbol ScottoKeebs:Placeholder_Resistor
- added R3: 1k, Resistor_SMD:R_0201_0603Metric, symbol Device:R
- added R4, R5: 27.4, Resistor_SMD:R_0201_0603Metric, symbol Device:R
- added R8, R9: 5.1k, Resistor_SMD:R_0201_0603Metric, symbol Device:R
- added SWBOOT1: Switch, Button_Switch_SMD:SW_Push_1P1T_NO_CK_KSC6xxG, symbol ScottoKeebs:Placeholder_Switch
- added U1: W25Q128JVS, Package_SO:SOIC-8_5.3x5.3mm_P1.27mm, symbol Memory_Flash:W25Q128JVS
- added U2: RP2040, Package_DFN_QFN:QFN-56-1EP_7x7mm_P0.4mm_EP3.2x3.2mm, symbol MCU_RaspberryPi:RP2040
- added U3: DWM1001, RF_Module:DecaWave_DWM1001, symbol RF_Module:DWM1001
- added YABM8-272-T1: Crystal_GND24, Oscillator:XTAL_ABM8-272-T3, symbol Device:Crystal_GND24
- C1, C2: value 1nF -> 15p
- C10, C11, C13: value 2.93 -> 100n
- C12: value 1.0uF -> 100n
- C14: value 2.92 -> 100n
- C15: value 2.2nF -> 100n
- C3, C4, C6, C8: value 1nF -> 100n
- C5, C7: value 1nF -> 1u
- C9: value 1nF -> 10u
Connections:
- net GND: now also C10.2, C11.2, C3.2, C4.2, C5.2, C6.2, C7.2, C8.2, C9.2, H27.1, H28.1, J1.A1 (GND_A), J1.A12 (GND_A__1), J1.B1 (GND_B), J1.B12 (GND_B__1), J1.SH1 (SHIELD), J1.SH2 (SHIELD__1), J1.SH3 (SHIELD__2), J1.SH4 (SHIELD__3), R8.1, R9.2, SWBOOT1.1, U1.4 (GND), U2.57 (GND), U3.1 (GND), U3.11 (GND), U3.24 (GND), U3.34 (GND), YABM8-272-T1.2, YABM8-272-T1.4; no longer C10.1, C11.1, C3.1, C4.1, C5.1, C6.1, C7.1, C8.1, C9.1
- net at H22.1: now also U2.37 (GPIO25)
- net at H9.1: now also U2.15 (GPIO12)
- net at H2.1: now also U2.7 (GPIO5)
- net at H13.1: now also U2.27 (GPIO16)
- net at H1.1: now also U2.6 (GPIO4)
- net at H23.1: now also U2.38 (GPIO26_ADC0)
- net at H20.1: now also U2.35 (GPIO23)
- net at H26.1: now also U2.41 (GPIO29_ADC3)
- net at H5.1: now also U2.11 (GPIO8)
- net +3.3V: now reaches C12.1, C15.1
- net +3.3V: now also C10.1, C11.1, C13.1, C14.1, C6.1, C7.1, C8.1, C9.1, H4.1, R1.2, R2.2, U1.8 (VCC), U2.1 (IOVDD), U2.10 (IOVDD), U2.22 (IOVDD), U2.33 (IOVDD), U2.42 (IOVDD), U2.43 (ADC_AVDD), U2.44 (VREG_IN), U2.48 (USB_VDD), U2.49 (IOVDD), U3.12 (VCC)
- net at H14.1: now also U2.28 (GPIO17)
- net at H16.1: now also U2.30 (GPIO19)
- net at H24.1: now also U2.39 (GPIO27_ADC1)
- net at H6.1: now also U2.12 (GPIO9)
- net at H7.1: now also U2.13 (GPIO10)
- net at H8.1: now also U2.14 (GPIO11)
- net at H15.1: now also U2.29 (GPIO18)
- net at H17.1: now also U2.31 (GPIO20)
- net at H18.1: now also U2.32 (GPIO21)
- net at H25.1: now also U2.40 (GPIO28_ADC2)
- net at H11.1: now also U2.17 (GPIO14)
- net at H12.1: now also U2.18 (GPIO15)
- net at H19.1: now also U2.34 (GPIO22)
- net at H21.1: now also U2.36 (GPIO24)
- net at H10.1: now also U2.16 (GPIO13)
- net at H3.1: now also U2.8 (GPIO6)
- removed net VDD: C1.2, C2.2, C3.2, C4.2, C5.2, C6.2, C7.2, C8.2
- new net: J1.A5 (CC1), R8.2
- new net: C2.2, U2.21 (XOUT), YABM8-272-T1.1
- new net: C1.2, U2.20 (XIN), YABM8-272-T1.3
- new net: R5.2, U2.46 (USB_DM)
- new net: J1.B5 (CC2), R9.1
- new net: R4.2, U2.47 (USB_DP)
- new net: R3.1, SWBOOT1.2
- new net +1V1: C3.1, C4.1, C5.1, R2.1, U2.23 (DVDD), U2.45 (VREG_VOUT), U2.50 (DVDD)
- new net +5V: J1.A4 (VBUS_A), J1.A9 (VBUS_A__1), J1.B4 (VBUS_B), J1.B9 (VBUS_B__1), R1.1
- new net DM: J1.A7 (DN1), J1.B7 (DN2), R5.1
- new net DP: J1.A6 (DP1), J1.B6 (DP2), R4.1
- new net QSPI_SCLK: U1.6 (CLK), U2.52 (QSPI_SCLK)
- new net QSPI_SD0: U1.5 (DI/IO_{0}), U2.53 (QSPI_SD0)
- new net QSPI_SD1: U1.2 (DO/IO_{1}), U2.55 (QSPI_SD1)
- new net QSPI_SD2: U1.3 (~{WP}/IO_{2}), U2.54 (QSPI_SD2)
- new net QSPI_SD3: U1.7 (~{HOLD}/~{RESET}/IO_{3}), U2.51 (QSPI_SD3)
- new net QSPI_SS: R3.2, U1.1 (~{CS}), U2.56 (QSPI_SS)
- new net RX: U2.2 (GPIO0), U3.26 (SPIS_MISO)
- new net csn: U2.3 (GPIO1), U3.29 (~{SPIS_CS})
- new net sck: U2.4 (GPIO2), U3.28 (SPIS_CLK)
- new net tx: U2.5 (GPIO3), U3.27 (SPIS_MOSI)
