File: marker.kicad_pcb (KiCad board)
At the start: 4 copper layers, 39.5 x 160 mm, 68 parts, among them J1 USB_A, U4 nRF5340-QKxx, Y2 Crystal

Commit message: doing the things
Parts:
- removed C16: 4.7uF, Capacitor_SMD:C_0201_0603Metric
- removed C17: 0.7F, Capacitor_SMD:C_0201_0603Metric
- removed H29, H30, H31, H32, H33, H34, H35, H36, H37, H38, H39, H40, H41, H42, H43, H44, H45, H46: MountingHole_Pad, MountingHole:MountingHole_2.5mm_Pad_Via
- removed L1: L, Inductor_SMD:L_6.3x6.3_H3
- removed U4: nRF5340-QKxx, Package_DFN_QFN:Nordic_AQFN-94-1EP_7x7mm_P0.4mm
- removed Y2: Crystal, Crystal:Crystal_SMD_3215-2Pin_3.2x1.5mm
- added G***: LOGO, LOGO, F.Cu at (117.0, 86.5)
- added R2: 2.2, Resistor_SMD:R_0201_0603Metric, F.Cu at (111.2, 78.2)
- added R3: 1k, Resistor_SMD:R_0201_0603Metric, F.Cu at (121.5, 83.8)
- added R4: 27.4, Resistor_SMD:R_0201_0603Metric, F.Cu at (120.2, 93.5)
- added R5: 27.4, Resistor_SMD:R_0201_0603Metric, F.Cu at (115.8, 122.5)
- added R8: 5.1k, Resistor_SMD:R_0201_0603Metric, F.Cu at (113.4, 123.5)
- added R9: 5.1k, Resistor_SMD:R_0201_0603Metric, F.Cu at (117.9, 123.4)
- added SWBOOT1: Switch, Button_Switch_SMD:SW_Push_1P1T_NO_CK_KSC6xxG, F.Cu at (120.0, 89.0)
- added U1: W25Q128JVS, Package_SO:SOIC-8_5.3x5.3mm_P1.27mm, F.Cu at (117.8, 80.1)
- added U2: RP2040, Package_DFN_QFN:QFN-56-1EP_7x7mm_P0.4mm_EP3.2x3.2mm, F.Cu at (115.2, 70.5)
- added U3: DWM1001, RF_Module:DecaWave_DWM1001, F.Cu at (114.5, 49.5)
- added YABM8-272-T1: Crystal_GND24, Oscillator:XTAL_ABM8-272-T3, F.Cu at (115.8, 61.6)
- C1, C2: value 1nF -> 15p
- C10, C11, C13: value 2.93 -> 100n
- C12: value 1.0uF -> 100n
- C14: value 2.92 -> 100n
- C15: value 2.2nF -> 100n
- C3, C4, C6, C8: value 1nF -> 100n
- C5, C7: value 1nF -> 1u
- C9: value 1nF -> 10u
- J1: value USB_A -> 2216100001; footprint Connector_USB:USB_A_Receptacle_GCT_USB1046 -> Connector_USB:MOLEX_2216100001
- R1: value 2R2 -> 1.7; footprint Resistor_SMD:R_01005_0402Metric -> Resistor_SMD:R_0201_0603Metric
- moved H6 114.7 mm to (98.0, 77.7)
- moved H5 114.4 mm to (98.0, 71.2)
- moved H4 114.0 mm to (98.0, 64.8)
- moved H8 108.8 mm to (98.0, 90.5)
- moved H7 103.9 mm to (98.0, 84.1)
- moved H24 97.0 mm to (130.8, 71.2), turned to 180 degrees
- moved J1 85.7 mm to (115.3, 132.2), turned to 0 degrees
- moved H23 83.8 mm to (130.8, 77.7), turned to 180 degrees
- moved H22 70.6 mm to (130.8, 84.1), turned to 180 degrees
- moved H9 59.2 mm to (98.0, 96.9)
- moved H10 58.9 mm to (98.0, 103.4)
- moved H11 58.6 mm to (98.0, 109.8)
- moved H12 42.3 mm to (98.0, 116.2)
- moved H13 42.1 mm to (98.0, 122.7)
- moved H14 41.9 mm to (98.0, 129.1)
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Connections:
- C1 pad 2: VDD -> Net-(U2-XIN)
- C10 pad 1: GND -> +3.3V
- C10 pad 2: Net-(U4-NFC1/P0.02) -> GND
- C11 pad 1: GND -> +3.3V
- C11 pad 2: Net-(U4-NFC1/P0.02) -> GND
- C12 pad 1: Net-(U4-DECR) -> +3.3V
- C13 pad 1: Net-(U4-NFC1/P0.02) -> +3.3V
- C14 pad 1: Net-(U4-NFC1/P0.02) -> +3.3V
- C15 pad 1: Net-(U4-DECR) -> +3.3V
- C2 pad 2: VDD -> Net-(U2-XOUT)
- C3 pad 1: GND -> +1V1
- C3 pad 2: VDD -> GND
- C4 pad 1: GND -> +1V1
- C4 pad 2: VDD -> GND
- C5 pad 1: GND -> +1V1
- C5 pad 2: VDD -> GND
- C6 pad 1: GND -> +3.3V
- C6 pad 2: VDD -> GND
- C7 pad 1: GND -> +3.3V
- C7 pad 2: VDD -> GND
- C8 pad 1: GND -> +3.3V
- C8 pad 2: VDD -> GND
- C9 pad 1: GND -> +3.3V
- C9 pad 2: Net-(U4-DECD) -> GND
- H27 pad 1: Net-(U4-AIN6/P0.27) -> GND
- H28 pad 1: Net-(U4-AIN7/P0.28) -> GND
- H4 pad 1: Net-(U4-AIN0/P0.04) -> +3.3V
- R1 pad 1: +5VD -> +5V
- R1 pad 2: magic -> +3.3V
Routing:
- net GND: track 0.00 -> 344.4 mm, vias 0 -> 13
- net Net-(U2-GPIO15): track 0.00 -> 169.8 mm, vias 0 -> 1
- net Net-(U2-GPIO10): track 0.00 -> 168.2 mm, vias 0 -> 15
- net +3.3V: track 0.00 -> 163.7 mm, vias 0 -> 7
- net Net-(U2-GPIO19): track 0.00 -> 128.1 mm, vias 0 -> 3
- net Net-(U2-GPIO22): track 0.00 -> 126.3 mm, vias 0 -> 3
- net Net-(U2-GPIO24): track 0.00 -> 125.1 mm, vias 0 -> 2
- net Net-(U2-GPIO14): track 0.00 -> 108.8 mm, vias 0 -> 1
- net Net-(U2-GPIO6): track 0.00 -> 102.3 mm, vias 0 -> 7
- net Net-(U2-GPIO25): track 0.00 -> 92.6 mm, vias 0 -> 3
- net Net-(U2-GPIO20): track 0.00 -> 92.1 mm, vias 0 -> 3
- net Net-(U2-GPIO23): track 0.00 -> 90.0 mm, vias 0 -> 6
- net Net-(U2-GPIO17): track 0.00 -> 83.4 mm, vias 0 -> 1
- net Net-(U2-GPIO9): track 0.00 -> 83.2 mm, vias 0 -> 4
- net Net-(U2-GPIO12): track 0.00 -> 82.4 mm, vias 0 -> 3
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Other:
- board size 39.5 x 160 mm -> 39.5 x 94 mm
- board text added: "10"
- board text added: "11"
- board text added: "12"
- board text added: "13"
- board text added: "14"
- board text added: "15"
- board text added: "16"
- board text added: "17"
- board text added: "18"
- board text added: "19"
- board text added: "20"
- board text added: "21"
- board text added: "22"
- board text added: "23"
- board text added: "24"
- board text added: "25"
- board text added: "3.3V"
- board text added: "4"
- board text added: "5"
- board text added: "6"
- board text added: "8"
- board text added: "9"
- board text added: "ADC 0"
- board text added: "ADC 1"
- board text added: "ADC 3"
- board text added: "ADC2"
- board text added: "BOOT"
- board text added: "GND"

Commit message: fab stuff
Parts:
- G***: moved to B.Cu
